File: Hardware/Timer Gate/Timer Gate/Timer Gate.sch (KiCad schematic (older format))
At the start: 5 parts, among them J1 OUTPUT, J2 SENSOR, U1 Trinket

Commit message: Updated course gate PCB, and updated the strobe code
Parts:
- J1: footprint Connectors2:1X02 -> Connectors2:1X03; symbol SparkFun-Connectors:CONN_02 -> SparkFun-Connectors:CONN_03
Connections:
- net at J2.1, U1.10 (+USB): now also J1.3
Changed lines of the file:
@@
 $EndComp
 $Comp
-L SparkFun-Connectors:CONN_02 J1
+L SparkFun-Connectors:CONN_03 J1
 U 1 1 5CD6E4CC
 P 4250 3400
-F 0 "J1" H 4206 3810 45  0000 C CNN
-F 1 "OUTPUT" H 4206 3726 45  0000 C CNN
-F 2 "Connectors2:1X02" H 4250 3650 20  0001 C CNN
+F 0 "J1" H 4200 3900 45  0000 C CNN
+F 1 "OUTPUT" H 4200 3800 45  0000 C CNN
+F 2 "Connectors2:1X03" H 4250 3650 20  0001 C CNN
 F 3 "" H 4250 3400 50  0001 C CNN
-F 4 "OUTPUT" H 4206 3631 60  0000 C CNN "Field4"
+F 4 "OUTPUT" H 4200 3700 60  0000 C CNN "Field4"
 	1    4250 3400
 	1    0    0    -1
@@
 	6350 4450 6350 4250
 Wire Wire Line
-	6350 4250 6250 4250
-Wire Wire Line
 	5100 4450 6350 4450
 Wire Wire Line
@@
 Wire Wire Line
 	4650 3850 5250 3850
+Wire Wire Line
+	6450 3850 6450 3200
+Connection ~ 6450 3850
+Wire Wire Line
+	6450 3200 4350 3200
+Wire Wire Line
+	6350 4250 6250 4250
 $EndSCHEMATC
